File: power.kicad_sch (KiCad schematic)
At the start: 16 parts, among them J1 USB_C, J2 batt conn., SW1 SW_Wuerth_450301014042, U3 TP4056-42-ESOP8, U4 AMS1117-3.3

Commit message: verder gewerkt aan pcb
Parts:
- added C103, C104: 10uf, Capacitor_SMD:C_0805_2012Metric, symbol Device:C
- added U5: MT3608, Package_TO_SOT_SMD:SOT-23-6, symbol Regulator_Switching:MT3608
Connections:
- net GND: now also U3.9 (EPAD), C103.2, C104.2
- net 3.3 v output renamed +3.3V
- net +3.3V: now also C103.1
- net 5v output: no longer names the net of SW1.3 (A)
- net 5v output: no longer U4.3 (VI)
- net battery output 5v renamed battery output
- net battery output: no longer SW1.1 (B)
- new net: C104.1, U4.3 (VI)
- no-connect marks 2 -> 3
Other:
- moved on the sheet: SW1, U4
